File: Kicad/esp/esp.kicad_sch (KiCad schematic)
At the start: 26 parts, among them J1 Conn_01x19_Pin, J2 Conn_01x19_Pin, P1 USB_C_Plug_USB2.0, Q1 NPN, Q2 NPN, SW1 SW_Push, SW2 SW_Push, U1 CH340C, U2 AMS1117-3.3, U3 ESP32-WROOM-E

Commit message: Shemat esp
Parts:
- removed C1: 0.01µ, symbol Device:C
- removed Q1, Q2: NPN, symbol Simulation_SPICE:NPN
- removed U1: CH340C, Package_SO:SOIC-16_3.9x9.9mm_P1.27mm, symbol Interface_USB:CH340C
- added C2, C5: 0.1µ, Capacitor_SMD:C_0805_2012Metric_Pad1.18x1.45mm_HandSolder, symbol Device:C
- added D1: LED_TX_Bleu, LED_SMD:LED_0805_2012Metric_Pad1.15x1.40mm_HandSolder, symbol Device:LED
- added D2: LED_RX_Rouge, LED_SMD:LED_0805_2012Metric_Pad1.15x1.40mm_HandSolder, symbol Device:LED
- added D3: D_Schottky, Diode_SMD:D_0805_2012Metric_Pad1.15x1.40mm_HandSolder, symbol Device:D_Schottky
- added J10: Sensor_car_out, Connector_PinHeader_2.54mm:PinHeader_1x03_P2.54mm_Vertical, symbol Connector_Generic:Conn_01x03
- added J11: Sensor_gate_open, Connector_PinHeader_2.54mm:PinHeader_1x03_P2.54mm_Vertical, symbol Connector_Generic:Conn_01x03
- added J12: Sensor_gate_close, Connector_PinHeader_2.54mm:PinHeader_1x03_P2.54mm_Vertical, symbol Connector_Generic:Conn_01x03
- added J3: LED_R, Connector_PinHeader_2.54mm:PinHeader_1x02_P2.54mm_Vertical, symbol Connector_Generic:Conn_01x02
- added J4: LED_V, Connector_PinHeader_2.54mm:PinHeader_1x02_P2.54mm_Vertical, symbol Connector_Generic:Conn_01x02
- added J5: SW_Open, Connector_PinHeader_2.54mm:PinHeader_1x02_P2.54mm_Vertical, symbol Connector_Generic:Conn_01x02
- added J6: SW_Close, Connector_PinHeader_2.54mm:PinHeader_1x02_P2.54mm_Vertical, symbol Connector_Generic:Conn_01x02
- added J7: Relay_gate_open, Connector_PinHeader_2.54mm:PinHeader_1x02_P2.54mm_Vertical, symbol Connector_Generic:Conn_01x02
- added J8: Sensor_car_in, Connector_PinHeader_2.54mm:PinHeader_1x03_P2.54mm_Vertical, symbol Connector_Generic:Conn_01x03
- added J9: Relay_gate_close, Connector_PinHeader_2.54mm:PinHeader_1x02_P2.54mm_Vertical, symbol Connector_Generic:Conn_01x02
- added Q1, Q2: NPN, Package_TO_SOT_SMD:SOT-23, symbol Transistor_BJT:BC846
- added R5, R6: 330, Resistor_SMD:R_0805_2012Metric_Pad1.20x1.40mm_HandSolder, symbol Device:R
- added U2: FT232RL, Package_SO:SSOP-28_5.3x10.2mm_P0.65mm, symbol Interface_USB:FT232RL
- C1: renamed from C2; footprint (none) -> Capacitor_SMD:C_0805_2012Metric_Pad1.18x1.45mm_HandSolder
- C3, C4: footprint (none) -> Capacitor_SMD:C_0805_2012Metric_Pad1.18x1.45mm_HandSolder
- C6: renamed from C5; footprint (none) -> Capacitor_SMD:C_0805_2012Metric_Pad1.18x1.45mm_HandSolder
- C7: renamed from C6; footprint (none) -> Capacitor_SMD:C_0805_2012Metric_Pad1.18x1.45mm_HandSolder
- J1, J2: footprint (none) -> Connector_PinHeader_2.54mm:PinHeader_1x19_P2.54mm_Vertical
- P1: footprint (none) -> Connector_USB:USB_C_Receptacle_GCT_USB4105-xx-A_16P_TopMnt_Horizontal
- R1: renamed from R3; footprint (none) -> Resistor_SMD:R_0805_2012Metric_Pad1.20x1.40mm_HandSolder
- R10: renamed from R8; footprint (none) -> Resistor_SMD:R_0805_2012Metric_Pad1.20x1.40mm_HandSolder
- R11: renamed from R9; footprint (none) -> Resistor_SMD:R_0805_2012Metric_Pad1.20x1.40mm_HandSolder
- R12: renamed from R10; footprint (none) -> Resistor_SMD:R_0805_2012Metric_Pad1.20x1.40mm_HandSolder
- R2: renamed from R4; footprint (none) -> Resistor_SMD:R_0805_2012Metric_Pad1.20x1.40mm_HandSolder
- R3: renamed from R5; value 1K -> 150; footprint (none) -> Resistor_SMD:R_0805_2012Metric_Pad1.20x1.40mm_HandSolder
- R4: renamed from R6; value 1K -> 150; footprint (none) -> Resistor_SMD:R_0805_2012Metric_Pad1.20x1.40mm_HandSolder
- R7: renamed from R1; footprint (none) -> Resistor_SMD:R_0805_2012Metric_Pad1.20x1.40mm_HandSolder
- R8: renamed from R2; footprint (none) -> Resistor_SMD:R_0805_2012Metric_Pad1.20x1.40mm_HandSolder
- R9: renamed from R7; footprint (none) -> Resistor_SMD:R_0805_2012Metric_Pad1.20x1.40mm_HandSolder
- SW1, SW2: footprint (none) -> Button_Switch_SMD:SW_SPST_CK_RS282G05A3
- renumbered U2 to U1
Connections:
- net +3.3V: now also C5.1, R5.2, R6.2
- net +5V: now also J1.19 (Pin_19), C2.1, D3.1 (K), U2.20 (VCC); no longer J1.18 (Pin_18), P1.A4 (VBUS), P1.A9 (VBUS), P1.B4 (VBUS), P1.B9 (VBUS)
- net D+: now also U2.15 (USBD+)
- net D-: now also U2.16 (USBD-)
- net DTR: now also Q2.2 (E)
- net EN: now also Q1.3 (C)
- net GND: now also C2.2, C5.2, U2.18 (GND), U2.21 (GND), U2.25 (AGND), U2.26 (TEST), U2.7 (GND)
- net IO0: now also Q2.3 (C)
- net RST: now also Q1.2 (E), U2.3 (RTS)
- net at C4.1: now also U2.2 (DTR)
- net at R3.1: now also U2.1 (TXD)
- net at R4.1: now also U2.5 (RXD)
- net at R7.2: now also Q1.1 (B)
- net at R8.2: now also Q2.1 (B)
- new net: D3.2 (A), P1.A4 (VBUS), P1.A9 (VBUS), P1.B4 (VBUS), P1.B9 (VBUS)
- new net: U2.17 (3V3OUT), U2.4 (VCCIO)
- new net: D2.1 (K), U2.22 (CBUS1)
- new net: D1.1 (K), U2.23 (CBUS0)
- new net: D2.2 (A), R6.1
- new net: D1.2 (A), R5.1
- no-connect marks 13 -> 18
Other:
- moved on the sheet: C1, C3, C4, C6, J1, J2, R1, R11, R12, R2, R3, R4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

Commit message: Kicad Final
Parts:
- removed J7: Relay_gate_open, Connector_PinHeader_2.54mm:PinHeader_1x02_P2.54mm_Vertical, symbol Connector_Generic:Conn_01x02
- removed J9: Relay_gate_close, Connector_PinHeader_2.54mm:PinHeader_1x02_P2.54mm_Vertical, symbol Connector_Generic:Conn_01x02
- added J1, J2: ~, TerminalBlock:TerminalBlock_bornier-2_P5.08mm, symbol Connector:Screw_Terminal_01x02
- added K1, K2: FINDER-30.22, Relay_THT:Relay_DPDT_Finder_30.22, symbol Relay:FINDER-30.22
- added R11, R12, R13, R15, R17: 10K, Resistor_SMD:R_0805_2012Metric_Pad1.20x1.40mm_HandSolder, symbol Device:R
- added R14, R20: 300, Resistor_SMD:R_0805_2012Metric_Pad1.20x1.40mm_HandSolder, symbol Device:R
- added R3, R4: 220, Resistor_SMD:R_0805_2012Metric_Pad1.20x1.40mm_HandSolder, symbol Device:R
- added U3: ULN2003, Package_SO:SO-16_3.9x9.9mm_P1.27mm, symbol Transistor_Array:ULN2003
- renumbered J12 to J10, J1 to J11, J2 to J12, J5 to J4, J8 to J5, J11 to J6, J4 to J7, J6 to J8, J10 to J9, R7 to R1, R2 to R10, R11 to R16, R9 to R18, R10 to R19, R8 to R2, R12 to R21, R3 to R5, R4 to R6, R5 to R7, R6 to R8, R1 to R9, U3 to U4
Connections:
- net +3.3V: now also R11.1, R12.1, R13.1, R15.1, R17.1, U3.9 (COM)
- net +5V: now also J10.1 (Pin_1), J5.1 (Pin_1), J6.1 (Pin_1), J9.1 (Pin_1), K1.A1, K2.A1
- net GND: now also J10.2 (Pin_2), J3.2 (Pin_2), J4.2 (Pin_2), J5.2 (Pin_2), J6.2 (Pin_2), J7.2 (Pin_2), J8.2 (Pin_2), J9.2 (Pin_2), U3.8 (GND)
- net IO15: now also R4.1
- net IO16: now also J6.3 (Pin_3), R11.2
- net IO17: now also J10.3 (Pin_3), R15.2
- net IO18: now also J9.3 (Pin_3), R17.2
- net IO19: now also J8.1 (Pin_1)
- net IO21: now also J4.1 (Pin_1), R12.2
- net IO22: now also R14.1
- net IO23: now also R20.1
- net IO4: now also R3.1
- net IO5: now also J5.3 (Pin_3), R13.2
- net at J3.1 (Pin_1): now also R14.2
- net at J7.1 (Pin_1): now also R20.2
- new net: J1.1 (Pin_1), K1.24, K2.11
- new net: J2.2 (Pin_2), K1.14, K2.14
- new net: J2.1 (Pin_1), K1.21, K2.21
- new net: J1.2 (Pin_2), K1.11, K2.24
- new net: K2.A2, U3.15 (O2)
- new net: K1.A2, U3.16 (O1)
- new net: R3.2, U3.14 (O3), U3.2 (I2), U3.4 (I4)
- new net: R4.2, U3.1 (I1), U3.13 (O4), U3.3 (I3)
- no-connect marks 18 -> 28
Other:
- moved on the sheet: C1, C2, C3, C4, C6, C7, D1, D2, J10, J11, J12, J7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

Commit message: MAJ Schema
Parts:
- removed J8: SW_Close, Connector_PinHeader_2.54mm:PinHeader_1x02_P2.54mm_Vertical, symbol Connector_Generic:Conn_01x02
- added R22, R23: 5.1K, Resistor_SMD:R_0805_2012Metric_Pad1.20x1.40mm_HandSolder, symbol Device:R
- P1: symbol Connector:USB_C_Plug_USB2.0 -> Connector:USB_C_Receptacle_USB2.0
Connections:
- net D+: now also P1.B6 (D+)
- net D-: now also P1.B7 (D-)
- net GND: now also R22.2, R23.2
- net at P1.A5 (CC1): now also R23.1
- net at P1.B5 (CC2): now also R22.1
Changed lines of the file:
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@@
   (junction (at 137.16 158.75) (diameter 0) (color 0 0 0 0)
   )
+  (junction (at 275.59 125.73) (diameter 0) (color 0 0 0 0)
+  )
   (junction (at 226.06 153.67) (diameter 0) (color 0 0 0 0)
   )
@@
   (junction (at 49.53 120.65) (diameter 0) (color 0 0 0 0)
   )
-  (junction (at 207.01 27.94) (diameter 0) (color 0 0 0 0)
-  )
   (junction (at 58.42 147.32) (diameter 0) (color 0 0 0 0)
   )
@@
   (no_connect (at 26.67 101.6))
   (no_connect (at 83.82 157.48))
-  (no_connect (at 265.43 107.95))
   (no_connect (at 270.51 67.31))
+  (no_connect (at 265.43 130.81))
   (no_connect (at 63.5 160.02))
   (no_connect (at 67.31 81.28))
@@
   (no_connect (at 67.31 106.68))
   (no_connect (at 63.5 162.56))
-  (no_connect (at 265.43 105.41))
+  (no_connect (at 265.43 128.27))
   (no_connect (at 246.38 67.31))
   (no_connect (at 26.67 91.44))
@@
     (stroke (width 0) (type default))
   )
+  (wire (pts (xy 279.4 125.73) (xy 275.59 125.73))
+    (stroke (width 0) (type default))
+  )
   (wire (pts (xy 54.61 27.94) (xy 59.69 27.94))
     (stroke (width 0) (type default))
@@
     (stroke (width 0) (type default))
   )
+  (wire (pts (xy 271.78 125.73) (xy 275.59 125.73))
+    (stroke (width 0) (type default))
+  )
   (wire (pts (xy 20.32 120.65) (xy 20.32 109.22))
     (stroke (width 0) (type default))
@@
     (stroke (width 0) (type default))
   )
+  (wire (pts (xy 265.43 107.95) (xy 271.78 107.95))
+    (stroke (width 0) (type default))
+  )
   (wire (pts (xy 160.02 27.94) (xy 170.18 27.94))
     (stroke (width 0) (type default))
@@
     (stroke (width 0) (type default))
   )
+  (wire (pts (xy 271.78 107.95) (xy 271.78 114.3))
+    (stroke (width 0) (type default))
+  )
   (wire (pts (xy 72.39 71.12) (xy 76.2 71.12))
     (stroke (width 0) (type default))
@@
     (stroke (width 0) (type default))
   )
+  (wire (pts (xy 265.43 105.41) (xy 279.4 105.41))
+    (stroke (width 0) (type default))
+  )
   (wire (pts (xy 219.71 132.08) (xy 226.06 132.08))
     (stroke (width 0) (type default))
@@
     (stroke (width 0) (type default))
   )
-  (wire (pts (xy 207.01 27.94) (xy 209.55 27.94))
-    (stroke (width 0) (type default))
-  )
   (wire (pts (xy 152.4 118.11) (xy 149.86 118.11))
     (stroke (width 0) (type default))
@@
     (stroke (width 0) (type default))
   )
+  (wire (pts (xy 279.4 105.41) (xy 279.4 114.3))
+    (stroke (width 0) (type default))
+  )
   (wire (pts (xy 269.24 85.09) (xy 269.24 86.36))
     (stroke (width 0) (type default))
@@
     (stroke (width 0) (type default))
   )
-  (wire (pts (xy 207.01 21.59) (xy 207.01 27.94))
+  (wire (pts (xy 279.4 121.92) (xy 279.4 125.73))
     (stroke (width 0) (type default))
   )
@@
     (stroke (width 0) (type default))
   )
+  (wire (pts (xy 265.43 118.11) (xy 265.43 120.65))
+    (stroke (width 0) (type default))
+  )
   (wire (pts (xy 149.86 50.8) (xy 149.86 63.5))
     (stroke (width 0) (type default))
@@
     (stroke (width 0) (type default))
   )
-  (wire (pts (xy 207.01 27.94) (xy 207.01 40.64))
+  (wire (pts (xy 207.01 21.59) (xy 207.01 40.64))
     (stroke (width 0) (type default))
   )
@@
     (stroke (width 0) (type default))
   )
+  (wire (pts (xy 271.78 121.92) (xy 271.78 125.73))
+    (stroke (width 0) (type default))
+  )
   (wire (pts (xy 246.38 24.13) (xy 248.92 24.13))
     (stroke (width 0) (type default))
@@
     (stroke (width 0) (type default))
   )
+  (wire (pts (xy 265.43 113.03) (xy 265.43 115.57))
+    (stroke (width 0) (type default))
+  )
   (label "IO5" (at 182.88 83.82 0) (fields_autoplaced)
     (effects (font (size 1.27 1.27)) (justify left bottom))
@@
   (label "D-" (at 265.43 113.03 0) (fields_autoplaced)
     (effects (font (size 1.27 1.27)) (justify left bottom))
+    (property "USB" "Default" (at 265.43 114.3 0)
+      (effects (font (size 1.27 1.27) italic) (justify left) hide)
+    )
   )
   (label "D+" (at 26.67 81.28 180) (fields_autoplaced)
@@
   (label "D+" (at 265.43 118.11 0) (fields_autoplaced)
     (effects (font (size 1.27 1.27)) (justify left bottom))
+    (property "USB" "Default" (at 265.43 119.38 0)
+      (effects (font (size 1.27 1.27) italic) (justify left) hide)
+    )
   )
   (label "IO35" (at 116.84 96.52 180) (fields_autoplaced)
@@
     (effects (font (size 1.27 1.27)) (justify right bottom))
   )
-  (label "IO19" (at 209.55 25.4 180) (fields_autoplaced)
-    (effects (font (size 1.27 1.27)) (justify right bottom))
-  )
   (label "IO13" (at 116.84 83.82 180) (fields_autoplaced)
     (effects (font (size 1.27 1.27)) (justify right bottom))
@@
     (effects (font (size 1.27 1.27)) (justify left bottom))
   )
+  (netclass_flag "" (length 2.54) (shape round) (at 265.43 114.3 270) (fields_autoplaced)
+    (effects (font (size 1.27 1.27)) (justify right bottom))
+    (property "USB" "" (at 267.97 113.6015 90)
+      (effects (font (size 1.27 1.27) italic) (justify left))
+    )
+  )
+  (netclass_flag "" (length 2.54) (shape round) (at 265.43 119.38 270) (fields_autoplaced)
+    (effects (font (size 1.27 1.27)) (justify right bottom))
+    (property "USB" "" (at 267.97 118.6815 90)
+      (effects (font (size 1.27 1.27) italic) (justify left))
+    )
+  )
   (symbol (lib_id "Connector:Conn_01x19_Pin") (at 265.43 46.99 0) (unit 1)
     (in_bom yes) (on_board yes) (dnp no)
@@
     )
   )
-  (symbol (lib_id "Connector_Generic:Conn_01x02") (at 214.63 25.4 0) (unit 1)
-    (in_bom yes) (on_board yes) (dnp no) (fields_autoplaced)
-    (property "Reference" "J8" (at 217.17 26.035 0)
-      (effects (font (size 1.27 1.27)) (justify left))
-    )
-    (property "Value" "SW_Close" (at 217.17 28.575 0)
-      (effects (font (size 1.27 1.27)) (justify left))
-    )
-    (property "Footprint" "Connector_PinHeader_2.54mm:PinHeader_1x02_P2.54mm_Vertical" (at 214.63 25.4 0)
-      (effects (font (size 1.27 1.27)) hide)
-    )
-    (property "Datasheet" "~" (at 214.63 25.4 0)
-      (effects (font (size 1.27 1.27)) hide)
-    )
-    (pin "1")
-    (pin "2")
-    (instances
-      (project "esp"
-        (path "/de08de6e-bdc7-4ddb-8300-6a16eecac9a6"
-          (reference "J8") (unit 1)
-        )
-      )
-    )
-  )
   (symbol (lib_id "power:+3.3V") (at 248.92 24.13 0) (unit 1)
     (in_bom yes) (on_board yes) (dnp no) (fields_autoplaced)
@@
     )
   )
+  (symbol (lib_id "Device:R") (at 271.78 118.11 0) (unit 1)
+    (in_bom yes) (on_board yes) (dnp no)
+    (property "Reference" "R22" (at 273.05 115.57 0)
+      (effects (font (size 1.27 1.27)) (justify left))
+    )
+    (property "Value" "5.1K" (at 273.05 118.11 0)
+      (effects (font (size 1.27 1.27)) (justify left))
+    )
+    (property "Footprint" "Resistor_SMD:R_0805_2012Metric_Pad1.20x1.40mm_HandSolder" (at 270.002 118.11 90)
+      (effects (font (size 1.27 1.27)) hide)
+    )
+    (property "Datasheet" "~" (at 271.78 118.11 0)
+      (effects (font (size 1.27 1.27)) hide)
+    )
+    (pin "1")
+    (pin "2")
+    (instances
+      (project "esp"
+        (path "/de08de6e-bdc7-4ddb-8300-6a16eecac9a6"
+          (reference "R22") (unit 1)
+        )
+      )
+    )
+  )
   (symbol (lib_id "Device:R") (at 199.39 124.46 90) (unit 1)
     (in_bom yes) (on_board yes) (dnp no) (fields_autoplaced)
@@
     )
   )
+  (symbol (lib_id "Device:R") (at 279.4 118.11 0) (unit 1)
+    (in_bom yes) (on_board yes) (dnp no)
+    (property "Reference" "R23" (at 280.67 115.57 0)
+      (effects (font (size 1.27 1.27)) (justify left))
+    )
+    (property "Value" "5.1K" (at 280.67 118.11 0)
+      (effects (font (size 1.27 1.27)) (justify left))
+    )
+    (property "Footprint" "Resistor_SMD:R_0805_2012Metric_Pad1.20x1.40mm_HandSolder" (at 277.622 118.11 90)
+      (effects (font (size 1.27 1.27)) hide)
+    )
+    (property "Datasheet" "~" (at 279.4 118.11 0)
+      (effects (font (size 1.27 1.27)) hide)
+    )
+    (pin "1")
+    (pin "2")
+    (instances
+      (project "esp"
+        (path "/de08de6e-bdc7-4ddb-8300-6a16eecac9a6"
+          (reference "R23") (unit 1)
+        )
+      )
+    )
+  )
   (symbol (lib_id "power:GND") (at 134.62 58.42 0) (unit 1)
     (in_bom yes) (on_board yes) (dnp no) (fields_autoplaced)
@@
     )
   )
+  (symbol (lib_id "power:GND") (at 275.59 125.73 0) (unit 1)
+    (in_bom yes) (on_board yes) (dnp no) (fields_autoplaced)
+    (property "Reference" "#PWR039" (at 275.59 132.08 0)
+      (effects (font (size 1.27 1.27)) hide)
+    )
+    (property "Value" "GND" (at 275.59 130.81 0)
+      (effects (font (size 1.27 1.27)))
+    )
+    (property "Footprint" "" (at 275.59 125.73 0)
+      (effects (font (size 1.27 1.27)) hide)
+    )
+    (property "Datasheet" "" (at 275.59 125.73 0)
+      (effects (font (size 1.27 1.27)) hide)
+    )
+    (pin "1")
+    (instances
+      (project "esp"
+        (path "/de08de6e-bdc7-4ddb-8300-6a16eecac9a6"
+          (reference "#PWR039") (unit 1)
+        )
+      )
+    )
+  )
   (symbol (lib_id "Transistor_BJT:BC846") (at 44.45 171.45 0) (unit 1)
     (in_bom yes) (on_board yes) (dnp no) (fields_autoplaced)
@@
     )
   )
-  (symbol (lib_id "Connector:USB_C_Plug_USB2.0") (at 250.19 115.57 0) (unit 1)
+  (symbol (lib_id "Connector:USB_C_Receptacle_USB2.0") (at 250.19 115.57 0) (unit 1)
     (in_bom yes) (on_board yes) (dnp no) (fields_autoplaced)
     (property "Reference" "P1" (at 250.19 93.98 0)
@@
     (pin "A6")
     (pin "A7")
+    (pin "A8")
     (pin "A9")
     (pin "B1")
@@
     (pin "B4")
     (pin "B5")
+    (pin "B6")
+    (pin "B7")
+    (pin "B8")
     (pin "B9")
     (pin "S1")
